File: camera-flash.sch (KiCad schematic (older format))
At the start: 17 parts, among them J1 USB, J10 CAM, J8 CAM, J9 CAM, U1 STUSB4500, U2 AP2204R-3.3

Commit message: routing 50% done"
Parts:
- gave numbers to parts that had none: 1
Changed lines of the file:
@@
 P 5950 6200
 AR Path="/5EEC9ABE/5EE5DDE3" Ref="J?"  Part="1"
-AR Path="/5EE5DDE3" Ref="J?"  Part="1"
-F 0 "J?" H 6030 6242 50  0000 L CNN
+AR Path="/5EE5DDE3" Ref="J11"  Part="1"
+F 0 "J11" H 6030 6242 50  0000 L CNN
 F 1 "GND" H 6030 6151 50  0000 L CNN
 F 2 "otter:Screw_Terminal_6x6x6mm" H 5950 6200 50  0001 C CNN

Commit message: update
Connections:
- net D+: no longer names the net of J1.A6 (D+)
- net D+: no longer J1.B6 (D+)
- net D-: no longer names the net of J1.A7 (D-)
- net D-: no longer J1.B7 (D-)
Changed lines of the file:
@@
 	0    1    1    0
 $EndComp
-Wire Wire Line
-	2950 4050 2950 4150
-Wire Wire Line
-	2950 4250 2950 4350
 $Comp
 L power:GND #PWR0102
@@
 	1    0    0    -1
 $EndComp
-Text GLabel 2950 4100 2    50   Input ~ 0
-D-
-Text GLabel 2950 4300 2    50   Input ~ 0
-D+
 NoConn ~ 2950 4650
 NoConn ~ 2950 4750
