File: LED_DRIVER.sch (KiCad schematic (older format))
At the start: 54 parts, among them J2 LED_WW_A, J3 LED_WW_C, J4 LED_CW_A, J5 LED_CW_C, Q1 2N7002, Q2 2N7002, Q3 BC847, Q4 BC857, Q5 BC847, Q6 BC857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

Commit message: routing 50% done"
Parts:
- removed Q1, Q2: 2N7002, Package_TO_SOT_SMD:SOT-23, symbol Transistor_FET:2N7002
- added Q1, Q2: ONSC-NMOS-8_E, Package_SO:SO-8_3.9x4.9mm_P1.27mm, symbol otter:ONSC-NMOS-8_E
- D1, D2: footprint Diode_SMD:D_SMA -> Diode_SMD:D_SOD-123F
- R10, R9: footprint otter:R_0603 -> otter:R_0805
Connections:
- net WW_DIM: no longer R12.2, R8.1, U4.6 (CS)
- net at C17.1, D1.2 (A), J2.1 (Pin_1)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: now also Q1.1 (S), Q1.2 (S), Q1.3 (S)
- net at C17.2, J3.1 (Pin_1), R7.2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: now also Q1.5 (D), Q1.6 (D), Q1.7 (D), Q1.8 (D)
- net at R19.1: now also Q1.4 (G)
- net at C18.1, D2.2 (A), J4.1 (Pin_1)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: now also Q2.1 (S), Q2.2 (S), Q2.3 (S)
- net at C18.2, J5.1 (Pin_1), R10.1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: now also Q2.5 (D), Q2.6 (D), Q2.7 (D), Q2.8 (D)
- net at R20.1: now also Q2.4 (G)
- new net CW_DIM: R12.2, R8.1, U4.6 (CS)
Other:
- moved on the sheet: C24, C25, Q3, Q4, Q5, Q6, Q7, Q8, R19, R20, R21, R22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

Commit message: finished layout
Connections:
- net +3V3: now also RV2.1; no longer RV2.2
- net at R12.1: now also RV2.2; no longer RV2.3
Other:
- moved on the sheet: R12
Changed lines of the file:
@@
 Text GLabel 4500 5750 1    50   Input ~ 0
-CW_DIM
-Text GLabel 5500 6650 3    50   Input ~ 0
 CW_DIM
 $Comp
@@
 	1    5500 6300
 	1    0    0    -1
-$EndComp
-$Comp
-L Device:R_Small R12
-U 1 1 5EEE42EE
-P 5500 6550
-F 0 "R12" H 5442 6596 50  0000 R CNN
-F 1 "150k" H 5442 6505 50  0000 R CNN
-F 2 "otter:R_0603" H 5500 6550 50  0001 C CNN
-F 3 "~" H 5500 6550 50  0001 C CNN
-	1    5500 6550
-	1    0    0    -1
-$EndComp
-$Comp
-L power:+3.3V #PWR0131
-U 1 1 5EEE42F4
-P 5650 6300
-F 0 "#PWR0131" H 5650 6150 50  0001 C CNN
-F 1 "+3.3V" V 5665 6428 50  0000 L CNN
-F 2 "" H 5650 6300 50  0001 C CNN
-F 3 "" H 5650 6300 50  0001 C CNN
-	1    5650 6300
-	0    1    1    0
 $EndComp
 Wire Wire Line
@@
 	5500 2700 5500 2800
 Connection ~ 5500 2800
+$Comp
+L power:+3.3V #PWR0131
+U 1 1 5EEE42F4
+P 5500 6150
+F 0 "#PWR0131" H 5500 6000 50  0001 C CNN
+F 1 "+3.3V" H 5515 6323 50  0000 C CNN
+F 2 "" H 5500 6150 50  0001 C CNN
+F 3 "" H 5500 6150 50  0001 C CNN
+	1    5500 6150
+	1    0    0    -1
+$EndComp
+$Comp
+L Device:R_Small R12
+U 1 1 5EEE42EE
+P 5750 6300
+F 0 "R12" V 5946 6300 50  0000 C CNN
+F 1 "150k" V 5855 6300 50  0000 C CNN
+F 2 "otter:R_0603" H 5750 6300 50  0001 C CNN
+F 3 "~" H 5750 6300 50  0001 C CNN
+	1    5750 6300
+	0    -1   -1   0
+$EndComp
+Text GLabel 5850 6300 2    50   Input ~ 0
+CW_DIM
 $EndSCHEMATC

Commit message: initial commit #2
Parts:
- Q1, Q2: symbol otter:ONSC-NMOS-8_E -> camera-flash-rescue:ONSC-NMOS-8_E-otter
- R10, R9: value R_Small -> 0.4
- U3, U4: symbol otter:lm3406 -> camera-flash-rescue:lm3406-otter
Changed lines of the file:
@@
 $EndDescr
 $Comp
-L otter:lm3406 U3
+L camera-flash-rescue:lm3406-otter U3
 U 1 1 5EEE41A3
 P 3700 2600
@@
 P 4950 2950
 F 0 "R9" H 5009 2996 50  0000 L CNN
-F 1 "R_Small" H 5009 2905 50  0000 L CNN
+F 1 "0.4" H 5009 2905 50  0000 L CNN
 F 2 "otter:R_0805" H 4950 2950 50  0001 C CNN
 F 3 "~" H 4950 2950 50  0001 C CNN
@@
 	3200 2800 3250 2800
 $Comp
-L otter:lm3406 U4
+L camera-flash-rescue:lm3406-otter U4
 U 1 1 5EEE4255
 P 3700 5550
@@
 P 4950 5900
 F 0 "R10" H 5009 5946 50  0000 L CNN
-F 1 "R_Small" H 5009 5855 50  0000 L CNN
+F 1 "0.4" H 5009 5855 50  0000 L CNN
 F 2 "otter:R_0805" H 4950 5900 50  0001 C CNN
 F 3 "~" H 4950 5900 50  0001 C CNN
@@
 Cin (min) = (IF * ton) / ^Vin (max) = 5µF\n^Vin (max) = 100mV
 $Comp
-L otter:ONSC-NMOS-8_E Q2
+L camera-flash-rescue:ONSC-NMOS-8_E-otter Q2
 U 1 1 5EE8D31F
 P 5700 5450
+AR Path="/5EE8D31F" Ref="Q2"  Part="1"
+AR Path="/5EEC9ABE/5EE8D31F" Ref="Q2"  Part="1"
 F 0 "Q2" H 6070 5328 60  0000 L CNN
 F 1 "ONSC-NMOS-8_E" H 5050 5550 60  0000 L CNN
@@
 Connection ~ 5500 5750
 $Comp
-L otter:ONSC-NMOS-8_E Q1
+L camera-flash-rescue:ONSC-NMOS-8_E-otter Q1
 U 1 1 5EEA5B2C
 P 5700 2500
+AR Path="/5EEA5B2C" Ref="Q1"  Part="1"
+AR Path="/5EEC9ABE/5EEA5B2C" Ref="Q1"  Part="1"
 F 0 "Q1" H 6070 2378 60  0000 L CNN
 F 1 "ONSC-NMOS-8_E" H 5050 2600 60  0000 L CNN
