File: SIGNAL.sch (KiCad schematic (older format))
At the start: 23 parts, among them J6 IN, J7 OUT, SW1 out, SW2 invert, SW3 no_delay, U5 TLP2366, U6 74LVC1G86, U7 74HCT123

Commit message: routing 50% done"
Parts:
- D5: footprint Diode_SMD:D_SMA -> Diode_SMD:D_SOD-123F
Connections:
- net at D5.2 (A), U5.3 (Cathode): now also J6.2 (Pin_2); no longer J6.1 (Pin_1)
- net at R13.2: now also J6.1 (Pin_1); no longer J6.2 (Pin_2)
Other:
- moved on the sheet: J6
Changed lines of the file:
@@
 F 0 "D5" V 3354 3072 50  0000 R CNN
 F 1 "D" V 3445 3072 50  0000 R CNN
-F 2 "Diode_SMD:D_SMA" H 3400 3150 50  0001 C CNN
+F 2 "Diode_SMD:D_SOD-123F" H 3400 3150 50  0001 C CNN
 F 3 "~" H 3400 3150 50  0001 C CNN
 	1    3400 3150
@@
 L Connector_Generic_MountingPin:Conn_01x02_MountingPin J?
 U 1 1 5EEF0C6E
-P 2550 3200
+P 2550 3100
 AR Path="/5EEF0C6E" Ref="J?"  Part="1"
 AR Path="/5EECA601/5EEF0C6E" Ref="J6"  Part="1"
-F 0 "J6" H 2637 3022 50  0000 L CNN
-F 1 "IN" H 2637 3113 50  0000 L CNN
-F 2 "Connector_Molex:Molex_PicoBlade_53261-0271_1x02-1MP_P1.25mm_Horizontal" H 2550 3200 50  0001 C CNN
-F 3 "~" H 2550 3200 50  0001 C CNN
-	1    2550 3200
-	-1   0    0    1
+F 0 "J6" H 2637 2922 50  0000 L CNN
+F 1 "IN" H 2637 3013 50  0000 L CNN
+F 2 "Connector_Molex:Molex_PicoBlade_53261-0271_1x02-1MP_P1.25mm_Horizontal" H 2550 3100 50  0001 C CNN
+F 3 "~" H 2550 3100 50  0001 C CNN
+	1    2550 3100
+	-1   0    0    -1
 $EndComp
 Wire Wire Line
@@
 L power:GND #PWR?
 U 1 1 5EEF0C78
-P 2550 2900
+P 2550 3400
 AR Path="/5EEF0C78" Ref="#PWR?"  Part="1"
 AR Path="/5EECA601/5EEF0C78" Ref="#PWR0151"  Part="1"
-F 0 "#PWR0151" H 2550 2650 50  0001 C CNN
-F 1 "GND" H 2555 2727 50  0000 C CNN
-F 2 "" H 2550 2900 50  0001 C CNN
-F 3 "" H 2550 2900 50  0001 C CNN
-	1    2550 2900
-	-1   0    0    1
-$EndComp
-$Comp
+F 0 "#PWR0151" H 2550 3150 50  0001 C CNN
+F 1 "GND" H 2555 3227 50  0000 C CNN
+F 2 "" H 2550 3400 50  0001 C CNN
+F 3 "" H 2550 3400 50  0001 C CNN
+	1    2550 3400
+	1    0    0    -1
+$EndComp
+$Comp

Commit message: finished layout
Connections:
- net +3V3: now also RV4.3; no longer RV4.2
- net at R16.1: now also RV4.2; no longer RV4.3
Other:
- moved on the sheet: RV4
Changed lines of the file:
@@
 Connection ~ 5650 3550
-$Comp
-L Device:R_POT RV?
-U 1 1 5EEF0C2F
-P 5650 3000
-AR Path="/5EEF0C2F" Ref="RV?"  Part="1"
-AR Path="/5EECA601/5EEF0C2F" Ref="RV3"  Part="1"
-F 0 "RV3" H 5581 3046 50  0000 R CNN
-F 1 "100k" H 5581 2955 50  0000 R CNN
-F 2 "otter:SV01A103AEA01R00" H 5650 3000 50  0001 C CNN
-F 3 "~" H 5650 3000 50  0001 C CNN
-	1    5650 3000
-	1    0    0    -1
-$EndComp
 $Comp
 L Device:R_Small R?
@@
 AR Path="/5EEF0C5A" Ref="RV?"  Part="1"
 AR Path="/5EECA601/5EEF0C5A" Ref="RV4"  Part="1"
-F 0 "RV4" H 7781 2846 50  0000 R CNN
-F 1 "100k" H 7781 2755 50  0000 R CNN
+F 0 "RV4" V 7643 2800 50  0000 C CNN
+F 1 "100k" V 7734 2800 50  0000 C CNN
 F 2 "otter:SV01A103AEA01R00" H 7850 2800 50  0001 C CNN
 F 3 "~" H 7850 2800 50  0001 C CNN
 	1    7850 2800
-	1    0    0    -1
+	0    1    1    0
 $EndComp
 $Comp
@@
 	1    7850 3050
 	1    0    0    -1
-$EndComp
-$Comp
-L power:+3.3V #PWR?
-U 1 1 5EEF0C66
-P 8000 2800
-AR Path="/5EEF0C66" Ref="#PWR?"  Part="1"
-AR Path="/5EECA601/5EEF0C66" Ref="#PWR0150"  Part="1"
-F 0 "#PWR0150" H 8000 2650 50  0001 C CNN
-F 1 "+3.3V" V 8015 2928 50  0000 L CNN
-F 2 "" H 8000 2800 50  0001 C CNN
-F 3 "" H 8000 2800 50  0001 C CNN
-	1    8000 2800
-	0    1    1    0
 $EndComp
 $Comp
@@
 Wire Wire Line
 	5850 3950 5950 3950
+$Comp
+L Device:R_POT RV?
+U 1 1 5EEF0C2F
+P 5650 3000
+AR Path="/5EEF0C2F" Ref="RV?"  Part="1"
+AR Path="/5EECA601/5EEF0C2F" Ref="RV3"  Part="1"
+F 0 "RV3" H 5581 3046 50  0000 R CNN
+F 1 "100k" H 5581 2955 50  0000 R CNN
+F 2 "otter:SV01A103AEA01R00" H 5650 3000 50  0001 C CNN
+F 3 "~" H 5650 3000 50  0001 C CNN
+	1    5650 3000
+	1    0    0    -1
+$EndComp
+$Comp
+L power:+3.3V #PWR?
+U 1 1 5EEF0C66
+P 7700 2800
+AR Path="/5EEF0C66" Ref="#PWR?"  Part="1"
+AR Path="/5EECA601/5EEF0C66" Ref="#PWR0150"  Part="1"
+F 0 "#PWR0150" H 7700 2650 50  0001 C CNN
+F 1 "+3.3V" V 7715 2928 50  0000 L CNN
+F 2 "" H 7700 2800 50  0001 C CNN
+F 3 "" H 7700 2800 50  0001 C CNN
+	1    7700 2800
+	0    -1   -1   0
+$EndComp
 $EndSCHEMATC

Commit message: initial commit #2
Parts:
- U5: symbol otter:TLP2366 -> camera-flash-rescue:TLP2366-otter
Changed lines of the file:
@@
 $EndComp
 $Comp
-L otter:TLP2366 U?
+L camera-flash-rescue:TLP2366-otter U?
 U 1 1 5EEF0BAF
 P 3850 3150
